Commit message: Added uwb anchors and made the actor more real

File: packages/smart_cart_description/urdf/smart_cart.urdf.xacro (robot description, xacro)
@@ -22,4 +22,7 @@
   <material name="grey_sensor">
     <color rgba="0.6 0.6 0.6 1.0"/>
+  </material>
+  <material name="cyan_uwb">
+    <color rgba="0.0 1.0 1.0 1.0"/>
   </material>
   <!-- ================================================ -->
@@ -86,5 +89,4 @@
       <dynamics damping="0.01" friction="0.01"/>
     </joint>
-    <!-- Gazebo Harmonic: low lateral friction to simulate omni rollers -->
     <gazebo reference="${name}_wheel">
       <mu1>0.5</mu1>
@@ -95,9 +97,55 @@
     </gazebo>
   </xacro:macro>
-  <!-- 4 wheels: FL, FR, RL, RR -->
+  <!-- 4 wheels -->
   <xacro:omni_wheel name="front_left"  x=" 0.25" y=" 0.27" z="-0.10"/>
   <xacro:omni_wheel name="front_right" x=" 0.25" y="-0.27" z="-0.10"/>
   <xacro:omni_wheel name="rear_left"   x="-0.25" y=" 0.27" z="-0.10"/>
   <xacro:omni_wheel name="rear_right"  x="-0.25" y="-0.27" z="-0.10"/>
+  <!-- ================================================ -->
+  <!-- UWB ANCHOR MACRO                                 -->
+  <!-- 4 anchors at cart corners – visual only          -->
+  <!-- Real UWB trilateration handled by                -->
+  <!-- uwb_simulator_node.py using odometry data        -->
+  <!-- ================================================ -->
+  <xacro:macro name="uwb_anchor" params="name x y">
+    <link name="${name}_uwb_anchor">
+      <!-- Anchor housing – small grey box -->
+      <visual>
+        <geometry>
+          <box size="0.04 0.04 0.03"/>
+        </geometry>
+        <material name="grey_sensor"/>
+      </visual>
+      <!-- Cyan glow sphere – indicates active UWB signal -->
+      <visual>
+        <origin xyz="0 0 0.03" rpy="0 0 0"/>
+        <geometry>
+          <sphere radius="0.025"/>
+        </geometry>
+        <material name="cyan_uwb"/>
+      </visual>
+      <inertial>
+        <mass value="0.05"/>
+        <inertia ixx="0.00001" iyy="0.00001" izz="0.00001"
+                 ixy="0" ixz="0" iyz="0"/>
+      </inertial>
+    </link>
+    <joint name="${name}_uwb_joint" type="fixed">
+      <parent link="base_link"/>
+      <child  link="${name}_uwb_anchor"/>
+      <!-- Mounted at top corners of cart body -->
+      <origin xyz="${x} ${y} 0.19" rpy="0 0 0"/>
+    </joint>
+    <!-- Gazebo: make the glow emissive so it's visible -->
+    <gazebo reference="${name}_uwb_anchor">
+      <material>Gazebo/Cyan</material>
+    </gazebo>
+  </xacro:macro>
+  <!-- 4 UWB anchors at cart corners -->
+  <!-- FL = front-left, FR = front-right, RL = rear-left, RR = rear-right -->
+  <xacro:uwb_anchor name="uwb_fl" x=" 0.32" y=" 0.23"/>
+  <xacro:uwb_anchor name="uwb_fr" x=" 0.32" y="-0.23"/>
+  <xacro:uwb_anchor name="uwb_rl" x="-0.32" y=" 0.23"/>
+  <xacro:uwb_anchor name="uwb_rr" x="-0.32" y="-0.23"/>
   <!-- ================================================ -->
   <!-- 2D LIDAR – RPLIDAR A1                           -->
@@ -113,5 +161,6 @@
     <inertial>
       <mass value="0.17"/>
-      <inertia ixx="0.0001" iyy="0.0001" izz="0.0001" ixy="0" ixz="0" iyz="0"/>
+      <inertia ixx="0.0001" iyy="0.0001" izz="0.0001"
+               ixy="0" ixz="0" iyz="0"/>
     </inertial>
   </link>
@@ -121,5 +170,4 @@
     <origin xyz="0.25 0 0.20" rpy="0 0 0"/>
   </joint>
-  <!-- Gazebo Harmonic LiDAR sensor -->
   <gazebo reference="lidar_link">
     <sensor name="lidar" type="gpu_lidar">
@@ -164,5 +212,6 @@
     <inertial>
       <mass value="0.072"/>
-      <inertia ixx="0.0001" iyy="0.0001" izz="0.0001" ixy="0" ixz="0" iyz="0"/>
+      <inertia ixx="0.0001" iyy="0.0001" izz="0.0001"
+               ixy="0" ixz="0" iyz="0"/>
     </inertial>
   </link>
@@ -172,5 +221,4 @@
     <origin xyz="0.35 0 0.20" rpy="0 0.15 0"/>
   </joint>
-  <!-- Optical frame – required for correct image projection -->
   <link name="camera_optical_link"/>
   <joint name="camera_optical_joint" type="fixed">
@@ -179,5 +227,4 @@
     <origin xyz="0 0 0" rpy="-1.5708 0 -1.5708"/>
   </joint>
-  <!-- Gazebo Harmonic depth camera sensor -->
   <gazebo reference="camera_link">
     <sensor name="depth_camera" type="depth_camera">
@@ -194,8 +241,5 @@
           <format>R8G8B8</format>
         </image>
-        <clip>
-          <near>0.1</near>
-          <far>10.0</far>
-        </clip>
+        <clip><near>0.1</near><far>10.0</far></clip>
         <noise>
           <type>gaussian</type>
@@ -217,5 +261,6 @@
       <inertial>
         <mass value="0.009"/>
-        <inertia ixx="0.00001" iyy="0.00001" izz="0.00001" ixy="0" ixz="0" iyz="0"/>
+        <inertia ixx="0.00001" iyy="0.00001" izz="0.00001"
+                 ixy="0" ixz="0" iyz="0"/>
       </inertial>
     </link>
@@ -225,5 +270,4 @@
       <origin xyz="0.36 ${y_offset} 0.05" rpy="0 0 0"/>
     </joint>
-    <!-- Gazebo Harmonic: model ultrasonic as narrow GPU ray sensor -->
     <gazebo reference="${name}_us_link">
       <sensor name="${name}_ultrasonic" type="gpu_lidar">
@@ -274,5 +318,5 @@
     </plugin>
   </gazebo>
-  <!-- Joint state publisher plugin – Gazebo Harmonic -->
+  <!-- Joint state publisher plugin -->
   <gazebo>
     <plugin filename="gz-sim-joint-state-publisher-system"

Commit message: rViz follow-me part is complete.

File: packages/smart_cart_description/urdf/smart_cart.urdf.xacro (robot description, xacro)
@@ -55,5 +55,5 @@
     <parent link="base_footprint"/>
     <child  link="base_link"/>
-    <origin xyz="0 0 0.175" rpy="0 0 0"/>
+    <origin xyz="0 0 0.175" rpy="0 0 3.14159"/>
   </joint>
   <!-- ================================================ -->
@@ -302,6 +302,6 @@
     <plugin filename="gz-sim-diff-drive-system"
             name="gz::sim::systems::DiffDrive">
-      <left_joint>front_left_wheel_joint</left_joint>
-      <right_joint>front_right_wheel_joint</right_joint>
+      <left_joint>front_right_wheel_joint</left_joint>
+      <right_joint>front_left_wheel_joint</right_joint>
       <wheel_separation>0.54</wheel_separation>
       <wheel_radius>0.075</wheel_radius>

Commit message: Made changes to show all in rViz

File: packages/smart_cart_description/urdf/smart_cart.urdf.xacro (robot description, xacro)
@@ -31,4 +31,5 @@
   <link name="base_link">
     <visual>
+      <origin xyz="0 0 0" rpy="0 0 3.14159"/>
       <geometry>
         <box size="${cart_length} ${cart_width} ${cart_height}"/>
@@ -51,10 +52,10 @@
   </link>
   <!-- base_footprint for Nav2 compatibility -->
-  <link name="base_footprint"/>
+  <!-- <link name="base_footprint"/>
   <joint name="base_footprint_joint" type="fixed">
     <parent link="base_footprint"/>
     <child  link="base_link"/>
-    <origin xyz="0 0 0.175" rpy="0 0 3.14159"/>
-  </joint>
+    <origin xyz="0 0 0.175" rpy="0 0 0"/>
+  </joint> -->
   <!-- ================================================ -->
   <!-- OMNI WHEEL MACRO                                 -->
@@ -98,8 +99,8 @@
   </xacro:macro>
   <!-- 4 wheels -->
-  <xacro:omni_wheel name="front_left"  x=" 0.25" y=" 0.27" z="-0.10"/>
-  <xacro:omni_wheel name="front_right" x=" 0.25" y="-0.27" z="-0.10"/>
-  <xacro:omni_wheel name="rear_left"   x="-0.25" y=" 0.27" z="-0.10"/>
-  <xacro:omni_wheel name="rear_right"  x="-0.25" y="-0.27" z="-0.10"/>
+  <xacro:omni_wheel name="front_left"  x=" 0.25" y=" 0.27" z="-0.15"/>
+  <xacro:omni_wheel name="front_right" x=" 0.25" y="-0.27" z="-0.15"/>
+  <xacro:omni_wheel name="rear_left"   x="-0.25" y=" 0.27" z="-0.15"/>
+  <xacro:omni_wheel name="rear_right"  x="-0.25" y="-0.27" z="-0.15"/>
   <!-- ================================================ -->
   <!-- UWB ANCHOR MACRO                                 -->
@@ -231,5 +232,5 @@
       <gz_frame_id>camera_optical_link</gz_frame_id>
       <topic>camera</topic>
-      <update_rate>30</update_rate>
+      <update_rate>15</update_rate>
       <always_on>true</always_on>
       <visualize>false</visualize>
@@ -237,6 +238,6 @@
         <horizontal_fov>1.5708</horizontal_fov>
         <image>
-          <width>640</width>
-          <height>480</height>
+          <width>320</width>
+          <height>240</height>
           <format>R8G8B8</format>
         </image>
@@ -274,5 +275,5 @@
         <gz_frame_id>${name}_us_link</gz_frame_id>
         <topic>ultrasonic/${name}</topic>
-        <update_rate>40</update_rate>
+        <update_rate>10</update_rate>
         <always_on>true</always_on>
         <lidar>
@@ -313,5 +314,5 @@
       <topic>cmd_vel</topic>
       <odom_topic>odom</odom_topic>
-      <tf_topic>tf</tf_topic>
+      <tf_topic>/tf</tf_topic>
       <frame_id>odom</frame_id>
       <child_frame_id>base_link</child_frame_id>

Commit message: Added full functional follow me part

File: packages/smart_cart_description/urdf/smart_cart.urdf.xacro (robot description, xacro)
@@ -31,5 +31,6 @@
   <link name="base_link">
     <visual>
-      <origin xyz="0 0 0" rpy="0 0 3.14159"/>
+      <!-- <origin xyz="0 0 0" rpy="0 0 3.14159"/> -->
+      <origin xyz="0 0 0" rpy="0 0 0.0"/>
       <geometry>
         <box size="${cart_length} ${cart_width} ${cart_height}"/>
@@ -87,5 +88,5 @@
       <child  link="${name}_wheel"/>
       <origin xyz="${x} ${y} ${z}" rpy="1.5708 0 0"/>
-      <axis xyz="0 0 1"/>
+      <axis xyz="0 0 -1"/>
       <dynamics damping="0.01" friction="0.01"/>
     </joint>
@@ -303,6 +304,6 @@
     <plugin filename="gz-sim-diff-drive-system"
             name="gz::sim::systems::DiffDrive">
-      <left_joint>front_right_wheel_joint</left_joint>
-      <right_joint>front_left_wheel_joint</right_joint>
+      <left_joint>front_left_wheel_joint</left_joint>
+      <right_joint>front_right_wheel_joint</right_joint>
       <wheel_separation>0.54</wheel_separation>
       <wheel_radius>0.075</wheel_radius>
