Commit message: Final code edit before submision

File: smart_cart_design_vignesh/urdf/smart_cart_3.urdf (robot description, URDF)
Before this commit: robot smart_cart_3, 12 links, 11 joints
Joints:
- joint uwb_fl_joint: origin xyz=0.32 0.27 0.3 -> xyz=0.32 0.23 0.3
- joint uwb_fr_joint: origin xyz=0.32 -0.27 0.3 -> xyz=0.32 -0.23 0.3
- joint uwb_rl_joint: origin xyz=-0.32 0.27 0.3 -> xyz=-0.32 0.23 0.3
- joint uwb_rr_joint: origin xyz=-0.32 -0.27 0.3 -> xyz=-0.32 -0.23 0.3
